File: PCB/Keyboard_lowprofile.kicad_pcb (KiCad board)
At the start: 2 copper layers, 277.8 x 136.2 mm, 161 parts, among them J1 Conn_01x02_Socket, SW1 SW_SPDT_312, U1 Nice_Nano_V2

Commit message: Fixed routes added silkscreen checked if Nice!nano Fits
Parts:
- added G***: LOGO, logos_better:fue, F.Cu at (247.0, 129.5)
- added G***: LOGO, logos_better:mon, F.Cu at (147.0, 147.5)
- added G***: LOGO, logos_better:pika, F.Cu at (89.0, 140.0)
- added G***: LOGO, logos_better:pika, B.Cu at (249.6, 59.4)
- added G***: LOGO, logos_better:mon, B.Cu at (145.5, 48.5)
- added G***: LOGO, logos_better:fue, B.Cu at (38.5, 93.5)
Routing:
- net Column 8: track 380.7 -> 367.6 mm
- net Net-(D55-A): track 150.1 -> 150.7 mm
Other:
- outline, holes or cut-outs redrawn
